File: HoverPuck.sch (EAGLE design)
At the start: 47 parts, among them J2 1X4, U1 EFM8BB1.QFN20, U2 TPS62177.DQC, U3 LM2731.DBV, U4 BLE112-A

Commit message: Working on v1.1 Schematic almost complete, need to work on routing pins now. Decided to not be stingy and control the full H Brudge with two sets of PWMs instead of one. I have the pins, might as well.
Parts:
- removed C11, C12, C13, C14, C5, C6: 0.1uF, standardparts:CAPACITOR.0603
- removed J6, J7: (no value), solderjumper:SOLDERJUMPER.2.SML.PASTE
- removed MB0, MB1: 1X2, headers.edge(.1in):1X2
- removed TP3, TP4, TP5, TP6: TPTP06R, testpad:TPTP06R
- removed U5, U6: (no value), packages(ti):DRV8800.RTY
- added Q1, Q2, Q3, Q4: (no value), fairchild:FDMA
- added R2: 51k, standardparts:RESISTOR.0603
- added RA2: 1k, resistorarray:RA-4.0603
- added SJ1: (no value), solderjumper:SOLDERJUMPER.2.SML.PASTE
- J1: value (none) -> 1X4; device solderjumper:SOLDERJUMPER.2.SML.PASTE -> headers(2mm):1X4
- J2: device headers.edge(.1in):1X4 -> headers(2mm):1X4
- RA1: value (none) -> 1k
Connections:
- removed net 12V: C12.1, C13.1, C14.1, C5.1, U5.VMOT, U6.VMOT
- removed net 20V_EN: RA1.2.2, TP5.TP, U1.P0.0, U3.!SHDN
- removed net N$10: J6.1, U4.P0_4
- removed net N$11: J7.1, U4.P0_5
- removed net N$14: MB0.2, U5.OUT-
- removed net N$15: MB1.1, U6.OUT+
- removed net N$16: MB1.2, U6.OUT-
- removed net N$17: C6.1, U5.CP1
- removed net N$18: C6.2, U5.CP2
- removed net N$19: C11.2, U6.CP2
- removed net N$20: C11.1, U6.CP1
- new net MB0+: J2.1, Q1.A.S, Q2.B.D
- new net MB0-: J2.2, Q1.B.S, Q2.A.D
- new net MB1+: J2.3, Q3.A.S, Q4.B.D
- new net MB1-: J2.4, Q3.B.S, Q4.A.D
- new net PWM0+: Q1.A.G, Q2.A.G, RA2.2.2
- new net PWM0-: Q1.B.G, Q2.B.G, RA2.1.2
- new net PWM1+: Q3.A.G, Q4.A.G, RA2.4.2
- new net PWM1-: Q3.B.G, Q4.B.G, RA2.3.2
- net 1S_DBG: now also J1.3; no longer J2.3
- net 20V: now also Q1.A.D, Q1.B.D, Q3.A.D, Q3.B.D
- net 3.3V: no longer U5.ENABLE, U5.MODE, U6.ENABLE, U6.MODE
- net ADC0: now also SJ1.2; no longer J1.2
- net EN_20V: now also R2.2, RA1.2.2, U1.P0.0, U3.!SHDN; no longer U5.!SLEEP, U6.!SLEEP
- net GND: now also J1.4, Q2.A.S, Q2.B.S, Q4.A.S, Q4.B.S, RA2.1.1, RA2.2.1, RA2.3.1, RA2.4.1, U4.P0_2; no longer C13.2, C14.2, J2.4, TP6.TP, U5.GND, U5.SENSE, U6.GND, U6.SENSE
- net N$1: now also U1.P1.1; no longer C12.2, U6.VCP
- net N$12: now also SJ1.1; no longer J1.1
- net N$13: now also U1.P1.3; no longer MB0.1, U5.OUT+
- net N$2: now also U1.P1.2; no longer C5.2, U5.VCP
- net PWM0: no longer TP3.TP, U5.PHASE
- net PWM1: no longer TP4.TP, U6.PHASE
- net RXI: now also U4.P0_4; no longer J6.2
- net TXO: now also U4.P0_5; no longer J7.2
- net VBAT: now also J1.1, R2.1; no longer J2.1
Other:
- moved on the sheet: C7, J2

Commit message: HoverPuck v1.1 completed. Send to OSHPark and PCBWay
Parts:
- removed B1: (no value), alps:SKSCLDE010
- removed SJ1: (no value), solderjumper:SOLDERJUMPER.2.SML.PASTE
- removed TP1, TP2: TPTP06R, testpad:TPTP06R
- added S1: SKSLLAE010, alps:SKSLLAE010
Connections:
- removed net N$1: U1.P1.1
- removed net N$12: SJ1.1, U1.P0.1
- removed net N$13: U1.P1.3
- removed net N$2: U1.P1.2
- removed net PWM0: U1.P0.3
- removed net PWM1: U1.P0.6
- removed net STATUS: RA1.1.2, U1.P0.7
- new net STAT1: RA1.2.1, U1.P1.1
- new net STAT2: RA1.1.1, U1.P1.0
- net 20V: no longer TP2.TP
- net 3.3V: now also RA1.3.1, RA1.4.1; no longer RA1.3.2, RA1.4.2, TP1.TP
- net ADC0: now also U1.P0.0; no longer SJ1.2
- net BLE_!RST: now also RA1.4.2, U1.P1.2; no longer RA1.3.1, U1.P1.0
- net EFM8_C2CK: now also S1.1; no longer B1.3, B1.4
- net EN_20V: now also U1.P0.1; no longer RA1.2.2, U1.P0.0
- net GND: now also S1.2; no longer B1.1, B1.2
- net N$4: now also RA1.3.2; no longer RA1.4.1
- net N$8: now also D3.1, RA1.2.2; no longer D4.1, RA1.1.1
- net N$9: now also D4.1, RA1.1.2; no longer D3.1, RA1.2.1
- net PWM0+: now also RA2.1.2, U1.P0.6; no longer RA2.2.2
- net PWM0-: now also RA2.2.2, U1.P0.7; no longer RA2.1.2
- net PWM1+: now also RA2.3.2, U1.P0.3; no longer RA2.4.2
- net PWM1-: now also RA2.4.2, U1.P0.2; no longer RA2.3.2
Other:
- moved on the sheet: RA1.1, RA1.2, RA1.3, RA1.4, RA2.1, RA2.2, RA2.3, RA2.4
